File: Eagle_PCB/Prototype/RC_Engine_Sound_ESP32.brd (EAGLE design)
At the start: 80 x 59.7 mm, 88 parts, among them IC1 7805T, IC2 PAM8403, Q1 BC337-25, Q2 BC337-25, Q3 BC337-25, Q4 BC337-25, Q5 BC337-25, Q6 BC337-25, Q7 BC337-25, Q8 BC337-25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

Commit message: Solved board issues after assembling of first PCB
Parts:
- removed JP20: (no value), 00_custom_pinhead:1X02
- removed R27: 330R, rcl:0207/2V
- moved JP12 1.27 mm to (14.0, 3.81)
- moved Q2 1.27 mm to (14.0, 10.2)
- moved JP11 1.27 mm to (8.89, 3.81)
- moved Q1 1.27 mm to (8.89, 10.2)
- moved Q9 1.27 mm to (59.7, 7.62)
- moved C1 0.63 mm to (34.9, 29.2)
Connections:
- removed net D0: R13.1, R27.1, U1.D0
- removed net N$31: JP20.1, R27.2
- net D3: now also R13.1
- net GND: no longer JP20.2
Routing:
- net D3: track 2.54 -> 29.0 mm
- net D0: track 5.08 -> 0.00 mm
- net N$31: track 5.08 -> 0.00 mm
- net N$6: track 3.81 -> 5.08 mm
- net N$4: track 5.08 -> 6.35 mm
- net N$15: track 17.8 -> 16.5 mm
- net N$17: track 23.8 -> 22.6 mm
- net N$16: track 17.8 -> 17.1 mm
Other:
- board text added: "ESP32 RC Sound & Light Controller 30 Pin V1.1"
- board text removed: "ESP32 RC Sound & Light Controller"
