File: Eagle_PCB/Prototype/RC_Engine_Sound_ESP32.sch (EAGLE design)
At the start: 88 parts, among them IC1 7805T, IC2 PAM8403, Q1 BC337-25, Q2 BC337-25, Q3 BC337-25, Q4 BC337-25, Q5 BC337-25, Q6 BC337-25, Q7 BC337-25, Q8 BC337-25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

Commit message: Solved board issues after assembling of first PCB
Parts:
- removed JP20: (no value), 00_custom_pinhead:PINHD-1X2
- removed R27: 330R, rcl:R-EU_0207/2V
Connections:
- removed net D0: R13.1, R27.1, U1.IO0
- removed net N$31: JP20.1, R27.2
- net D3: now also R13.1
- net GND: no longer JP20.2
Other:
- note added: "Prototype board for 36 pin ESP32 V1.1"
- note added: "V1.1: - R3 faulty track repaired - Headlights moved from D0 to D3, caused boot issues - 5V plane removed below screw head areas"
- note removed: "Prototype board for 36 pin ESP32"
Changed lines of the file:
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@@
 <part name="R19" library="rcl" deviceset="R-EU_" device="0207/2V" value="47R"/>
 <part name="JP16" library="00_custom_pinhead" deviceset="PINHD-2X3" device=""/>
-<part name="JP20" library="00_custom_pinhead" deviceset="PINHD-1X2" device=""/>
-<part name="GND24" library="supply1" deviceset="GND" device=""/>
-<part name="R27" library="rcl" deviceset="R-EU_" device="0207/2V" value="330R"/>
 <part name="JP21" library="00_custom_pinhead" deviceset="PINHD-1X2" device=""/>
 <part name="GND25" library="supply1" deviceset="GND" device=""/>
@@
 <text x="15.24" y="233.68" size="1.778" layer="91">Battery input
 7.0 - 12.6V</text>
-<text x="292.1" y="27.94" size="3.048" layer="91">Prototype board for 36 pin ESP32</text>
+<text x="289.56" y="27.94" size="3.048" layer="91">Prototype board for 36 pin ESP32 V1.1</text>
 <text x="347.98" y="88.9" size="1.778" layer="91">Shaker motor</text>
 <text x="38.1" y="147.32" size="1.778" layer="91" rot="R90">Headlights</text>
@@
 LED can be wired directly, but don't have the full brightness!</text>
 <text x="10.16" y="68.58" size="1.778" layer="91">LED driver transistors. Never connect LED directly, always use a matching series resistor!</text>
+<text x="185.42" y="71.12" size="1.778" layer="91">V1.1:
+- R3 faulty track repaired
+- Headlights moved from D0 to D3, caused boot issues
+- 5V plane removed below screw head areas</text>
 </plain>
 <instances>
@@
 </instance>
 <instance part="JP16" gate="A" x="152.4" y="124.46" rot="R90"/>
-<instance part="JP20" gate="G$1" x="25.4" y="27.94"/>
-<instance part="GND24" gate="1" x="15.24" y="20.32"/>
-<instance part="R27" gate="G$1" x="15.24" y="40.64" rot="R270"/>
 <instance part="JP21" gate="G$1" x="45.72" y="27.94"/>
 <instance part="GND25" gate="1" x="35.56" y="20.32"/>
@@
 </segment>
 <segment>
-<pinref part="GND24" gate="1" pin="GND"/>
-<wire x1="15.24" y1="22.86" x2="15.24" y2="27.94" width="0.1524" layer="91"/>
-<pinref part="JP20" gate="G$1" pin="2"/>
-<wire x1="15.24" y1="27.94" x2="22.86" y2="27.94" width="0.1524" layer="91"/>
-</segment>
-<segment>
 <pinref part="GND25" gate="1" pin="GND"/>
 <wire x1="35.56" y1="22.86" x2="35.56" y2="27.94" width="0.1524" layer="91"/>
@@
 <wire x1="218.44" y1="45.72" x2="218.44" y2="48.26" width="0.1524" layer="91"/>
 <label x="218.44" y="48.26" size="1.778" layer="95" rot="R90" xref="yes"/>
+</segment>
+<segment>
+<pinref part="R13" gate="G$1" pin="1"/>
+<wire x1="20.32" y1="167.64" x2="20.32" y2="172.72" width="0.1524" layer="91"/>
+<label x="20.32" y="172.72" size="1.778" layer="95" rot="R90" xref="yes"/>
 </segment>
 </net>
@@
 </segment>
 </net>
-<net name="D0" class="0">
-<segment>
-<pinref part="U1" gate="G$1" pin="IO0"/>
-<wire x1="236.22" y1="127" x2="236.22" y2="121.92" width="0.1524" layer="91"/>
-<label x="236.22" y="121.92" size="1.778" layer="95" rot="R270" xref="yes"/>
-</segment>
-<segment>
-<pinref part="R13" gate="G$1" pin="1"/>
-<wire x1="20.32" y1="167.64" x2="20.32" y2="172.72" width="0.1524" layer="91"/>
-<label x="20.32" y="172.72" size="1.778" layer="95" rot="R90" xref="yes"/>
-</segment>
-<segment>
-<pinref part="R27" gate="G$1" pin="1"/>
-<wire x1="15.24" y1="45.72" x2="15.24" y2="48.26" width="0.1524" layer="91"/>
-<label x="15.24" y="48.26" size="1.778" layer="95" rot="R90" xref="yes"/>
-</segment>
-</net>
 <net name="N$17" class="0">
 <segment>
@@
 </segment>
 </net>
-<net name="N$31" class="0">
-<segment>
-<pinref part="JP20" gate="G$1" pin="1"/>
-<wire x1="22.86" y1="30.48" x2="15.24" y2="30.48" width="0.1524" layer="91"/>
-<pinref part="R27" gate="G$1" pin="2"/>
-<wire x1="15.24" y1="30.48" x2="15.24" y2="35.56" width="0.1524" layer="91"/>
-</segment>
-</net>
