File: Eagle_PCB/Final/RC_Engine_Sound_ESP32.sch (EAGLE design)
At the start: 84 parts, among them IC1 7805T, IC2 PAM8403, Q1 BC337-25, Q10 BC337-25, Q11 IRLZ44N, Q12 BC337-25, Q13 BC337-25, Q2 BC337-25, Q3 BC337-25, Q4 BC337-25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

Commit message: PCB v1.1: moved R28 away from trailer connector
Parts:
- R29: value 10k -> 4k7
Other:
- note added: "Board for 30 pin ESP32 V1.1"
- note removed: "Board for 30 pin ESP32"
Changed lines of the file:
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@@
 <part name="R31" library="rcl" deviceset="R-EU_" device="0207/2V" value="1k"/>
 <part name="GND29" library="supply1" deviceset="GND" device=""/>
-<part name="R29" library="rcl" deviceset="R-EU_" device="0207/2V" value="10k"/>
+<part name="R29" library="rcl" deviceset="R-EU_" device="0207/2V" value="4k7"/>
 <part name="JP32" library="00_custom_pinhead" deviceset="PINHD-1X3" device=""/>
 <part name="GND25" library="supply1" deviceset="GND" device=""/>
@@
 <text x="7.62" y="238.76" size="1.778" layer="91">Battery input
 7.0 - 12.6V</text>
-<text x="292.1" y="27.94" size="3.048" layer="91">Board for 30 pin ESP32</text>
+<text x="292.1" y="27.94" size="3.048" layer="91">Board for 30 pin ESP32 V1.1</text>
 <text x="347.98" y="88.9" size="1.778" layer="91">Shaker motor</text>
 <text x="170.18" y="91.44" size="1.778" layer="91" rot="R90">Headlights</text>
