File: Eagle_PCB/SMD/RC_Engine_Sound_ESP32.brd (EAGLE design)
At the start: 71.1 x 47 mm, 57 parts, among them IC1 7805DT, IC2 ULN2003AD, IC3 ULN2003AD, IC4 PAM8403_NO_SPEAKERS, U1 ESP32DEVKITV1

Commit message: v5.8: MAN TGX 680, SMD board v1.1
Parts:
- C1: value 1000uF -> 1000uF 10V; device rcl:E5-10,5 -> rcl:UD-10X10_NICHICON
- moved C1 0.45 mm to (11.7, 41.0), turned to 0 degrees
Routing:
- net GND: track 30.0 -> 43.0 mm, vias 9 -> 17
Other:
- board text added: "TheDIYGuy999 ESP32 RC Sound & Light Controller SMD 30 Pin V1.1"
- board text removed: "TheDIYGuy999 ESP32 RC Sound & Light Controller SMD 30 Pin V1.0"
